File: ursa.kicad_pcb (KiCad board)
At the start: 2 copper layers, 36 parts, among them SW10_L1 SW_Push, SW10_R1 SW_Push, SW11_L1 SW_Push, SW11_R1 SW_Push, SW12_L1 SW_Push, SW12_R1 SW_Push, SW13_L1 SW_Push, SW13_R1 SW_Push, SW14_L1 SW_Push, SW14_R1 SW_Push, SW15_L1 SW_Push, SW15_R1 SW_Push, SW16_L1 SW_Push, SW16_R1 SW_Push, SW17_L1 SW_Push, SW17_R1 SW_Push, SW1_L1 SW_Push, SW1_R1 SW_Push, SW2_L1 SW_Push, SW2_R1 SW_Push, SW3_L1 SW_Push, SW3_R1 SW_Push, SW4_L1 SW_Push, SW4_R1 SW_Push, SW5_L1 SW_Push, SW5_R1 SW_Push, SW6_L1 SW_Push, SW6_R1 SW_Push, SW7_L1 SW_Push, SW7_R1 SW_Push, SW8_L1 SW_Push, SW8_R1 SW_Push, SW9_L1 SW_Push, SW9_R1 SW_Push, U1_L1 WeAct-RP2040-Pico, U1_R1 WeAct-RP2040-Pico

Commit message: better wiring and through hole added
Parts:
- removed SW10_L1, SW10_R1, SW11_L1, SW11_R1, SW12_L1, SW12_R1, SW13_L1, SW13_R1, SW14_L1, SW14_R1, SW15_L1, SW15_R1, SW16_L1, SW16_R1, SW17_L1, SW17_R1, SW1_L1, SW1_R1, SW2_L1, SW2_R1, SW3_L1, SW3_R1, SW4_L1, SW4_R1, SW5_L1, SW5_R1, SW6_L1, SW6_R1, SW7_L1, SW7_R1, SW8_L1, SW8_R1, SW9_L1, SW9_R1: SW_Push, keyswitches:Kailh_socket_MX_optional
- removed U1_L1, U1_R1: WeAct-RP2040-Pico, WeAct-RP2040-Pico:WeAct-RP2040-Pico
- added HL_1: MountingHole, MountingHole:MountingHole_2.2mm_M2, F.Cu at (38.8, 98.2)
- added HL_2: MountingHole, MountingHole:MountingHole_2.2mm_M2, F.Cu at (34.5, 74.8)
- added HL_3: MountingHole, MountingHole:MountingHole_2.2mm_M2, F.Cu at (39.1, 40.1)
- added HL_4: MountingHole, MountingHole:MountingHole_2.2mm_M2, F.Cu at (124.8, 45.5)
- added HL_5: MountingHole, MountingHole:MountingHole_2.2mm_M2, F.Cu at (124.8, 106.8)
- added HL_6: MountingHole, MountingHole:MountingHole_2.2mm_M2, F.Cu at (78.8, 105.8)
- added HR_1: MountingHole, MountingHole:MountingHole_2.2mm_M2, F.Cu at (271.5, 98.2)
- added HR_2: MountingHole, MountingHole:MountingHole_2.2mm_M2, F.Cu at (277.2, 74.8)
- added HR_3: MountingHole, MountingHole:MountingHole_2.2mm_M2, F.Cu at (271.1, 41.1)
- added HR_4: MountingHole, MountingHole:MountingHole_2.2mm_M2, F.Cu at (230.7, 106.8)
- added HR_5: MountingHole, MountingHole:MountingHole_2.2mm_M2, F.Cu at (185.8, 106.8)
- added HR_6: MountingHole, MountingHole:MountingHole_2.2mm_M2, F.Cu at (185.9, 45.9)
- added JL_1: TRRS, Keebio:TRRS-PJ-320A, F.Cu at (149.8, 108.5)
- added JR_1: TRRS, Keebio:TRRS-PJ-320A, F.Cu at (160.8, 108.5)
- added SWL_1: SW_Push, keyswitches:Kailh_socket_MX_optional, F.Cu at (43.9, 53.0)
- added SWL_10: SW_Push, keyswitches:Kailh_socket_MX_optional, F.Cu at (111.3, 69.1)
- added SWL_11: SW_Push, keyswitches:Kailh_socket_MX_optional, F.Cu at (43.9, 85.3)
- added SWL_12: SW_Push, keyswitches:Kailh_socket_MX_optional, F.Cu at (60.6, 85.3)
- added SWL_13: SW_Push, keyswitches:Kailh_socket_MX_optional, F.Cu at (77.5, 85.3)
- added SWL_14: SW_Push, keyswitches:Kailh_socket_MX_optional, F.Cu at (94.4, 85.3)
- added SWL_15: SW_Push, keyswitches:Kailh_socket_MX_optional, F.Cu at (111.3, 85.3)
- added SWL_16: SW_Push, keyswitches:Kailh_socket_MX_optional, F.Cu at (111.3, 101.8)
- added SWL_17: SW_Push, keyswitches:Kailh_socket_MX_optional, F.Cu at (94.4, 101.8)
- added SWL_2: SW_Push, keyswitches:Kailh_socket_MX_optional, F.Cu at (60.6, 53.0)
- added SWL_3: SW_Push, keyswitches:Kailh_socket_MX_optional, F.Cu at (77.6, 53.0)
- added SWL_4: SW_Push, keyswitches:Kailh_socket_MX_optional, F.Cu at (94.5, 53.0)
- added SWL_5: SW_Push, keyswitches:Kailh_socket_MX_optional, F.Cu at (111.3, 53.0)
- added SWL_6: SW_Push, keyswitches:Kailh_socket_MX_optional, F.Cu at (43.9, 69.1)
- added SWL_7: SW_Push, keyswitches:Kailh_socket_MX_optional, F.Cu at (60.6, 69.1)
- added SWL_8: SW_Push, keyswitches:Kailh_socket_MX_optional, F.Cu at (77.6, 69.1)
- added SWL_9: SW_Push, keyswitches:Kailh_socket_MX_optional, F.Cu at (94.6, 69.0)
- added SWR_1: SW_Push, keyswitches:Kailh_socket_MX_optional, F.Cu at (199.0, 53.0)
- added SWR_10: SW_Push, keyswitches:Kailh_socket_MX_optional, F.Cu at (266.0, 69.2)
- added SWR_11: SW_Push, keyswitches:Kailh_socket_MX_optional, F.Cu at (199.0, 85.5)
- added SWR_12: SW_Push, keyswitches:Kailh_socket_MX_optional, F.Cu at (215.8, 85.5)
- added SWR_13: SW_Push, keyswitches:Kailh_socket_MX_optional, F.Cu at (232.5, 85.5)
- added SWR_14: SW_Push, keyswitches:Kailh_socket_MX_optional, F.Cu at (249.2, 85.5)
- added SWR_15: SW_Push, keyswitches:Kailh_socket_MX_optional, F.Cu at (266.0, 85.5)
- added SWR_16: SW_Push, keyswitches:Kailh_socket_MX_optional, F.Cu at (199.0, 101.8)
- added SWR_17: SW_Push, keyswitches:Kailh_socket_MX_optional, F.Cu at (215.8, 101.8)
- added SWR_2: SW_Push, keyswitches:Kailh_socket_MX_optional, F.Cu at (215.8, 53.0)
- added SWR_3: SW_Push, keyswitches:Kailh_socket_MX_optional, F.Cu at (232.5, 53.0)
- added SWR_4: SW_Push, keyswitches:Kailh_socket_MX_optional, F.Cu at (249.2, 53.0)
- added SWR_5: SW_Push, keyswitches:Kailh_socket_MX_optional, F.Cu at (266.0, 53.0)
- added SWR_6: SW_Push, keyswitches:Kailh_socket_MX_optional, F.Cu at (199.0, 69.2)
- added SWR_7: SW_Push, keyswitches:Kailh_socket_MX_optional, F.Cu at (215.8, 69.2)
- added SWR_8: SW_Push, keyswitches:Kailh_socket_MX_optional, F.Cu at (232.5, 69.2)
- added SWR_9: SW_Push, keyswitches:Kailh_socket_MX_optional, F.Cu at (249.2, 69.2)
- added UL_1: WeAct-RP2040-Pico, WeAct-RP2040-Pico:WeAct-RP2040-Pico, F.Cu at (141.0, 72.0)
- added UR_1: WeAct-RP2040-Pico, WeAct-RP2040-Pico:WeAct-RP2040-Pico, F.Cu at (169.5, 72.0)

Commit message: Worked on layout
* solder mask added
* some lines added (not 100% sure what is called) to break the two
* through-hole adjusted
* still need to work on design
Parts:
- moved HR_5 29.1 mm to (157.0, 102.2)
- moved HL_5 17.9 mm to (142.0, 102.2)
- moved HL_3 15.6 mm to (25.8, 48.2)
- moved HL_2 8.99 mm to (25.8, 76.8)
- moved HR_3 7.48 mm to (273.2, 48.2)
- moved JR_1 7.36 mm to (153.4, 108.5)
- moved HL_4 7.09 mm to (118.2, 48.2)
- moved SWL_11 6.15 mm to (37.8, 86.0)
- moved SWL_1 6.14 mm to (37.8, 52.5)
- moved SWL_6 6.12 mm to (37.8, 69.2)
- moved UL_1 6.02 mm to (135.0, 71.5)
- moved SWL_12 5.90 mm to (54.8, 86.0)
- moved SWL_2 5.89 mm to (54.8, 52.5)
- moved SWL_3 5.89 mm to (71.8, 52.5)
- moved SWL_9 5.87 mm to (88.8, 69.2)
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Routing:
- added copper zone on B.Cu, net GND_L
- added copper zone on B.Cu, net GND_R
Other:
- board outline added: 254.5 x 68 mm

Commit message: Right side layout adjustment
* now render shows split PCB, fixed an issue where the cut edge weren't
  set properly.
* render images added
* left side PCB adjusted little bit! Gave smoother edge on the right
  most parts but the TRRS and RP2040 side edge are still right angle.
  Still deciding what to do.
Parts:
- moved HR_1 6.00 mm to (273.2, 98.2)
Other:
- outline, holes or cut-outs redrawn
Changed lines of the file:
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@@
   )
   (footprint "MountingHole:MountingHole_2.2mm_M2" (layer "F.Cu")
-    (at 267.25 98.25)
+    (at 273.25 98.25)
     (descr "Mounting Hole 2.2mm, no annular, M2")
     (tags "mounting hole 2.2mm no annular m2")
@@
   (gr_line (start 25.75 44.75) (end 145.75 44.75) (layer "Edge.Cuts") (width 0.1))
   (gr_arc (start 229.25 109.25) (mid 228.224874 111.724874) (end 225.75 112.75) (layer "Edge.Cuts") (width 0.1))
-  (gr_line (start 229.5 101.75) (end 229.25 101.75) (layer "Edge.Cuts") (width 0.1))
   (gr_line (start 22.25 48.25) (end 22.25 101.75) (layer "Edge.Cuts") (width 0.1))
+  (gr_line (start 229.25 105.25) (end 229.25 109.25) (layer "Edge.Cuts") (width 0.1))
   (gr_arc (start 75.75 112.75) (mid 73.275126 111.724874) (end 72.25 109.25) (layer "Edge.Cuts") (width 0.1))
-  (gr_line (start 229.25 101.75) (end 229.25 109.25) (layer "Edge.Cuts") (width 0.1))
   (gr_arc (start 22.25 48.25) (mid 23.275126 45.775126) (end 25.75 44.75) (layer "Edge.Cuts") (width 0.1))
-  (gr_line (start 276.75 47.75) (end 276.75 76.25) (layer "Edge.Cuts") (width 0.1))
   (gr_line (start 153.25 112.75) (end 153.25 44.75) (layer "Edge.Cuts") (width 0.1))
   (gr_line (start 145.75 112.75) (end 75.75 112.75) (layer "Edge.Cuts") (width 0.1))
-  (gr_line (start 276.75 76.75) (end 276.75 101.75) (layer "Edge.Cuts") (width 0.1))
+  (gr_arc (start 229.25 105.25) (mid 230.275126 102.775126) (end 232.75 101.75) (layer "Edge.Cuts") (width 0.1))
+  (gr_line (start 232.75 101.75) (end 273.25 101.75) (layer "Edge.Cuts") (width 0.1))
   (gr_line (start 22.25 101.75) (end 72.25 101.75) (layer "Edge.Cuts") (width 0.1))
   (gr_arc (start 273.25 44.75) (mid 275.724874 45.775126) (end 276.75 48.25) (layer "Edge.Cuts") (width 0.1))
   (gr_line (start 145.75 44.75) (end 145.75 112.75) (layer "Edge.Cuts") (width 0.1))
   (gr_line (start 225.75 112.75) (end 153.25 112.75) (layer "Edge.Cuts") (width 0.1))
-  (gr_line (start 276.75 101.75) (end 229.5 101.75) (layer "Edge.Cuts") (width 0.1))
-  (gr_line (start 276.75 48.25) (end 276.75 76.75) (layer "Edge.Cuts") (width 0.1))
   (gr_line (start 72.25 101.75) (end 72.25 109.25) (layer "Edge.Cuts") (width 0.1))
+  (gr_line (start 276.75 48.25) (end 276.75 98.25) (layer "Edge.Cuts") (width 0.1))
   (gr_line (start 273.25 44.75) (end 153.25 44.75) (layer "Edge.Cuts") (width 0.1))
+  (gr_arc (start 276.75 98.25) (mid 275.724874 100.724874) (end 273.25 101.75) (layer "Edge.Cuts") (width 0.1))
   (zone (net 68) (net_name "GND_R") (layer "B.Cu") (hatch edge 0.508)
     (connect_pads (clearance 0.3))
@@
     (polygon
       (pts
-        (xy 281 101.75)
-        (xy 233.5 101.75)
-        (xy 233.5 112.75)
-        (xy 157.5 112.75)
-        (xy 157.5 44.5)
-        (xy 281 44.5)
+        (xy 275.5 44.75)
+        (xy 276 45)
+        (xy 276.75 45.75)
+        (xy 277.25 46.5)
+        (xy 277.25 99)
+        (xy 277 102.25)
+        (xy 232 102.25)
+        (xy 230.5 103.25)
+        (xy 229.75 104.75)
+        (xy 229.75 113.25)
+        (xy 153 113.25)
+        (xy 152.75 44.25)
+        (xy 274.75 44.25)
       )
     )
@@
     (polygon
       (pts
-        (xy 150 112.75)
-        (xy 76.5 112.75)
-        (xy 76.5 101.75)
-        (xy 26.5 101.75)
-        (xy 26.5 44.75)
-        (xy 150 44.75)
+        (xy 145.75 112.75)
+        (xy 72.25 112.75)
+        (xy 72.25 101.75)
+        (xy 22.25 101.75)
+        (xy 22.25 44.75)
+        (xy 145.75 44.75)
       )
     )
